File: DBJ/greenhousectrl.sch (EAGLE design)
At the start: 30 parts, among them IC1 ATMEGA168TQFP-08, IC3 7805DT, IC4 L298, J1 5.5x2.1mm Barrel, Y2 16MHZ

Commit message: rev 0.0.1 of schematic
first rev of full schematic capture
Parts:
- added D10: Zener, SparkFun-DiscreteSemi:DIODE-ZENER
- added D9: 1N4148, SparkFun-DiscreteSemi:DIODEKIT
- added J2: (no value), SparkFun-Connectors:M03SCREW
- added J3: (no value), SparkFun-Connectors:M03-SCREW-5MM
- added JP1: JUMPER-PAD-2-NOYES_SILK, SparkFun-Passives:JUMPER-PAD-2-NOYES_SILK
- added K1: JQX-15F, SparkFun-Electromechanical:RELAYPTH5
- added LED1: (no value), SparkFun-LED:LED5MM-KIT
- added Q1: 2N3904, SparkFun-DiscreteSemi:TRANSISTOR_NPN2N3904-EZ
- added R3, R4: 1K, SparkFun-Resistors:1KOHM-1/4W-1%(PTH)HORIZ-KIT
- added SV1: (no value), con-lsta:FE20-1
Connections:
- new net ADC4: SV1.4
- new net ADC5: SV1.5
- new net COIL: D10.C, JP1.1, K1.COIL2, Q1.C, R4.1
- new net COMMON: J3.3, K1.MAIN
- new net DIODENODE: D10.A, D9.A, JP1.2
- new net N$3: LED1.C, R4.2
- new net N$6: Q1.B, R3.1
- new net NC: J3.1, K1.NC
- new net NO: J3.2, K1.NO
- new net RELAY: J2.2, R3.2
- new net SS: SV1.11
- new net VCC: D9.C, J2.3, K1.COIL1, LED1.A
- net +5V: now also SV1.15, SV1.2
- net GND: now also J2.1, Q1.E, SV1.1, SV1.16, SV1.3
- net MISO: now also SV1.13
- net MOSI: now also SV1.12
- net SCK: now also SV1.14
