File: DBJ/greenhousectrl-lab.sch (EAGLE design)
At the start: 40 parts, among them IC1 ATMEGA168TQFP-08, IC3 7805DT, IC4 L298, J1 5.5x2.1mm Barrel, K1 JQX-15F, Q1 2N3904, Y2 16MHZ

Commit message: in-lab sync
Parts:
- removed PVAL1, PVAL2, SOIL-LEVEL, WATER-LEVEL: (no value), adafruit:JST_3PIN
- added D1, D11, D2, D3, D4, D5, D6, D7: (no value), adafruit:DIODESMA
Connections:
- removed net N$15: IC4.OUT2, X2-MOT2-1.KL
- removed net N$7: IC4.OUT1, X2-MOT2-2.KL
- removed net N$8: IC4.OUT3, X1-MOT1-2.KL
- removed net N$9: IC4.OUT4, X1-MOT1-1.KL
- new net N$20: D2.A
- new net OUT1: D1.A, D11.C, IC4.OUT1, X1-MOT1-1.KL
- new net OUT2: D2.C, D3.A, IC4.OUT2, X1-MOT1-2.KL
- new net OUT3: D4.C, D5.A, IC4.OUT3, X2-MOT2-1.KL
- new net OUT4: D6.C, D7.A, IC4.OUT4, X2-MOT2-2.KL
- net +12V: now also D1.C, D3.C, D5.C, D7.C
- net +5V: now also SL1.2, SL2.2, SL3.2, SL4.2; no longer PVAL1.2, PVAL2.2, SOIL-LEVEL.2, WATER-LEVEL.2
- net GND: now also D11.A, D4.A, D6.A, SL1.1, SL2.1, SL3.1, SL4.1; no longer PVAL1.3, PVAL2.3, SOIL-LEVEL.3, WATER-LEVEL.3
- net PC0: now also SL1.3; no longer PVAL1.1
- net PC1: now also SL2.3; no longer PVAL2.1
- net PC2: now also SL3.3; no longer SOIL-LEVEL.1
- net PC3: now also SL4.3; no longer WATER-LEVEL.1
Other:
- moved on the sheet: SL1, SL2, SL3, SL4, X1-MOT1-1, X1-MOT1-2, X2-MOT2-1, X2-MOT2-2
