File: DBJ/greenhousectrl-latest-monday-redo.sch (EAGLE design)
At the start: 56 parts, among them IC1 ATMEGA168TQFP-08, IC2 7824DT, IC4 L298, J1 POWER_JACKPTH, K2 G5LE, Q1 MMBT2222A, SW2 MOMENTARYBUTTON, X1 CRYSTALS-NOGND-HC49

Commit message: Replaced 1x20 LCD with 2 1x8, gerb and DRC checked
Parts:
- removed R10: (no value), adafruit:R-US_M0805
- removed SV1: (no value), con-lsta:FE20-1
- removed X2, X3, X4, X5: (no value), ece388:1X03_5MM_SCREW
- added J4, J5, J6, J7: (no value), SparkFun-Connectors:M03SCREW_LOCK
- added R15: 1k, adafruit:R-US_M0805
- added SV2, SV3: (no value), con-lsta:FE08-1
- C1, C2: value (none) -> 20pF
- R1, R2: value (none) -> 150
- R11, R8: value (none) -> 240
- R12, R7, R9: value (none) -> 1k
- R13: value (none) -> 3k
- R14: value (none) -> 1k; device SparkFun-Resistors:RESISTOR0402 -> adafruit:R-US_M0805
- R2(SMD), R5, R6: value (none) -> 10k
- R3: value 1K -> 1k
- R4: value 1K -> 150
Connections:
- removed net ADC4: SV1.4
- removed net ADC5: SV1.5
- removed net N$4: OK2.C, R7.2
- removed net N$9: OK1.C, R10.2
- removed net SS: SV1.11
- net +5V: now also J4.2, J5.2, J6.2, J7.2, R15.2, R7.2, SV2.7, SV3.2; no longer SV1.15, SV1.2, X2-2.KL, X3-2.KL, X4-2.KL, X5-2.KL
- net COMMON: now also J3.1; no longer J3.3
- net ENA: now also R7.1
- net ENB: now also R15.1
- net GND: now also J4.3, J5.3, J6.1, J7.1, OK1.C, OK2.C, SV2.6, SV2.8, SV3.1; no longer R10.1, R7.1, SV1.1, SV1.16, SV1.3, X2-1.KL, X3-1.KL, X4-3.KL, X5-3.KL
- net MISO: now also SV3.4; no longer SV1.13
- net MOSI: now also SV3.5; no longer SV1.12
- net NC: now also J3.2; no longer J3.1
- net NO: now also J3.3; no longer J3.2
- net PB2: now also SV3.6
- net PC0: now also J4.1; no longer X2-3.KL
- net PC1: now also J5.1; no longer X3-3.KL
- net PC2: now also J6.3; no longer X4-1.KL
- net PC3: now also J7.3; no longer X5-1.KL
- net PC4: now also SV2.5
- net PC5: now also SV2.4
- net SCK: now also SV3.3; no longer SV1.14
Other:
- moved on the sheet: R7
