File: DBJ/outdated/greenhousectrl-lab.sch (EAGLE design)
At the start: 30 parts, among them IC1 ATMEGA168TQFP-08, IC3 7805DT, IC4 L298, J1 5.5x2.1mm Barrel, Y2 16MHZ

Commit message: Updated Schematic Notes
smaller relay, smd parts added for leds instead of thru-hole, smaller
diodes for h-bridge
Parts:
- removed C1, C2: 0.1uF, SparkFun-Capacitors:0.1UF-25V(+80/-20%)(0603)
- removed CN1, CN2, CN3, CN4, PVAL1, PVAL2, SOIL-LEVEL, WATER-LEVEL: (no value), adafruit:JST_3PIN
- removed FRAME1: FRAME-LEDGER, SparkFun-Aesthetics:FRAME-LEDGER
- removed IC3: 7805DT, adafruit:7805DT
- added C6, C7: 0.1uF, SparkFun-Capacitors:0.1UF-25V(+80/-20%)(0603)
- added D1, D11, D2, D3, D4, D5, D6, D7: (no value), adafruit:DIODESOD-523
- added D10: Zener, adafruit:DIODESOD-323F
- added D9: 1N4148, adafruit:DIODESOD-323F
- added FTDI-SERIAL-HEADER: HEADER-06X1-MALE, GeekAmmo:HEADER-06X1-MALE
- added J3: (no value), SparkFun-Connectors:M03-SCREW-5MM
- added JP1: JUMPER-PAD-2-NOYES_SILK, SparkFun-Passives:JUMPER-PAD-2-NOYES_SILK
- added K1: RELAYPTH4, SparkFun-Electromechanical:RELAYPTH4
- added LED1: PL006-WCR13, led:PL006-WCR13
- added OK1, OK2: 4N27SM, optocoupler:4N27SM
- added Q1: MMBT2222A, SparkFun-DiscreteSemi:TRANSISTOR_NPNMMBT2222A
- added R10, R11, R12, R7, R8, R9: (no value), adafruit:R-US_M0805
- added R13, R14: (no value), SparkFun-Resistors:RESISTOR0402
- added R3, R4: 1K, adafruit:R-US_M0805
- added SL1, SL2, SL3, SL4: (no value), con-amp-quick:M03
- added SV1: (no value), con-lsta:FE20-1
- added U2: V_REG_317SMD, SparkFun-PowerIC:V_REG_317SMD
- renumbered ISP1 to ICSP-PROG-HEADER
Connections:
- net N$13 renamed SEN_A
- net N$14 renamed SEN_B
- removed net N$17: C4.1, ICSP-PROG-HEADER.RST
- new net ADC4: SV1.4
- new net ADC5: SV1.5
- new net COIL: D10.C, JP1.1, K1.COIL2, Q1.C, R4.1
- new net COMMON: J3.3, K1.MAIN
- new net CTS(DOESNTEXIST): FTDI-SERIAL-HEADER.2
- new net DIODENODE: D10.A, D9.A, JP1.2
- new net DTR: C4.1, FTDI-SERIAL-HEADER.6
- new net ENA: IC4.ENABLE_A, OK2.COL
- new net ENB: IC4.ENABLE_B, OK1.COL
- new net N$3: LED1.C, R4.2
- new net N$4: OK2.C, R7.2
- new net N$5: OK2.EMI, R9.2
- new net N$6: Q1.B, R3.1
- new net NC: J3.1, K1.NC
- new net NO: J3.2, K1.NO
- new net OUT1: D1.A, D11.C, IC4.OUT1, X1-MOT1-1.KL
- new net OUT2: D2.C, D3.A, IC4.OUT2, X1-MOT1-2.KL
- new net OUT3: D4.C, D5.A, IC4.OUT3, X2-MOT2-1.KL
- new net OUT4: D6.C, D7.A, IC4.OUT4, X2-MOT2-2.KL
- new net RST: C4.2, IC1.PC6(/RESET), ICSP-PROG-HEADER.RST, R2(SMD).1, SW1.P$1
- new net RX: FTDI-SERIAL-HEADER.5, IC1.PD0(RXD)
- new net SS: SV1.11
- new net TX: FTDI-SERIAL-HEADER.4, IC1.PD1(TXD)
- new net VCC: D9.C, K1.COIL1, LED1.A
- net +12V: now also C6.1, D1.C, D3.C, D5.C, D7.C, U2.IN; no longer C2.1, IC3.VI
- net +5V: now also C7.1, FTDI-SERIAL-HEADER.3, R14.2, SL1.2, SL2.2, SL3.2, SL4.2, SV1.15, SV1.2, U2.OUT; no longer C1.1, IC3.VO, PVAL1.2, PVAL2.2, SOIL-LEVEL.2, WATER-LEVEL.2
- net GND: now also C6.2, C7.2, D11.A, D2.A, D4.A, D6.A, FTDI-SERIAL-HEADER.1, OK1.BAS, OK2.BAS, Q1.E, R10.1, R12.1, R13.1, R7.1, R9.1, SL1.1, SL2.1, SL3.1, SL4.1, SV1.1, SV1.16, SV1.3; no longer C1.2, C2.2, IC3.GND, PVAL1.3, PVAL2.3, SOIL-LEVEL.3, WATER-LEVEL.3
- net MISO: now also SV1.13
- net MOSI: now also SV1.12
- net N$1: now also OK2.A, R8.2; no longer C4.2, IC1.PC6(/RESET), R2(SMD).1, SW1.P$1
- net N$15: now also OK1.EMI, R12.2; no longer IC4.OUT2, X2-MOT2-1.KL
- net N$7: now also R13.2, R14.1, U2.ADJ; no longer IC4.OUT1, X2-MOT2-2.KL
- net N$8: now also OK1.A, R11.2; no longer IC4.OUT3, X1-MOT1-2.KL
- net N$9: now also OK1.C, R10.2; no longer IC4.OUT4, X1-MOT1-1.KL
- net PB0: now also R3.2
- net PC0: now also SL1.3; no longer PVAL1.1
- net PC1: now also SL2.3; no longer PVAL2.1
- net PC2: now also SL3.3; no longer SOIL-LEVEL.1
- net PC3: now also SL4.3; no longer WATER-LEVEL.1
- net PD4: now also R8.1; no longer IC4.ENABLE_A
- net PD5: now also R11.1; no longer IC4.ENABLE_B
- net SCK: now also SV1.14
Other:
- note removed: "HBridge/Motor Controls"
- moved on the sheet: R5, R6, X1-MOT1-1, X1-MOT1-2, X2-MOT2-1, X2-MOT2-2
