File: DBJ/outdated/greenhousectrl-latest-monday-no-errors-fixed-cap.sch (EAGLE design)
At the start: 61 parts, among them IC1 ATMEGA168TQFP-08, IC2 7824DT, IC4 L298, J1 POWER_JACKPTH, K2 G5LE, Q1 MMBT2222A, SW2 MOMENTARYBUTTON, X1 CRYSTALS-NOGND-HC49, X6 1X03_35MM_SCREW, X7 1X03_35MM_SCREW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

Commit message: Replaced 1x20 LCD with 2 1x8, gerb and DRC checked
Parts:
- removed J2: (no value), SparkFun-Connectors:M03SCREW_LOCK
- removed R10: (no value), adafruit:R-US_M0805
- removed X2, X3, X4, X5: (no value), ece388:1X03_5MM_SCREW
- removed X6, X7, X8, X9: 1X03_35MM_SCREW, ece388:1X03_35MM_SCREW
- added J4, J5, J6, J7: (no value), SparkFun-Connectors:M03SCREW_LOCK
- added R15: 1k, adafruit:R-US_M0805
- C1, C2: value (none) -> 20pF
- R1, R2: value (none) -> 150
- R11, R8: value (none) -> 240
- R12, R14, R7, R9: value (none) -> 1k
- R13: value (none) -> 3k
- R2(SMD), R5, R6: value (none) -> 10k
- R4: value 1K -> 150
Connections:
- removed net N$4: OK2.C, R7.2
- removed net N$9: OK1.C, R10.2
- net +5V: now also J4.2, J5.2, J6.2, J7.2, R15.2, R7.2; no longer X2-2.KL, X3-2.KL, X4-2.KL, X5-2.KL
- net ENA: now also R7.1
- net ENB: now also R15.1
- net GND: now also J4.3, J5.3, J6.1, J7.1, OK1.C, OK2.C; no longer R10.1, R7.1, X2-1.KL, X3-1.KL, X4-3.KL, X5-3.KL
- net PC0: now also J4.1; no longer X2-3.KL
- net PC1: now also J5.1; no longer X3-3.KL
- net PC2: now also J6.3; no longer X4-1.KL
- net PC3: now also J7.3; no longer X5-1.KL
Other:
- moved on the sheet: R7
