File: pcb 2/production/friday-submit-ben/ghc-silk.brd (EAGLE design)
At the start: 73.6 x 70.8 mm, 59 parts, among them IC1 ATMEGA168TQFP-08, IC2 7805DT, IC4 L298, J1 POWER_JACKPTH, K2 G5LE, Q1 MMBT2222A, SW2 MOMENTARYBUTTON, U1 L298HEATSINK

Commit message: Fixed Traces
Routing:
- net N$7: track 91.3 -> 45.1 mm, vias 7 -> 2
- net PC5: track 51.5 -> 32.6 mm, vias 3 -> 2
- net +12V: track 141.7 -> 128.2 mm, vias 6 -> 5
- net PC4: track 43.9 -> 37.0 mm, vias 4 -> 2
- net +5V: track 309.5 -> 303.2 mm, vias 18 -> 16
- net VCC: track 22.3 -> 17.1 mm
- net MOSI: track 47.9 -> 45.4 mm
- net PB2: track 15.8 -> 14.4 mm, vias 2 -> 1
- net MISO: track 42.4 -> 43.6 mm
- net SCK: track 103.9 -> 102.7 mm, vias 4 -> 2
- net PD4: track 62.4 -> 61.6 mm
- net GND: track 43.0 -> 42.8 mm, vias 17 -> 18

Commit message: Replaced H-bridge, remapped pins where needed. Needs routing still
Parts:
- removed IC4: L298, st-microelectronics:MULTIWATT-15
Connections:
- removed net SEN_A: IC4.1, R5.1
- removed net SEN_B: IC4.15, R6.1
- new net ADC6: IC1.19, SV2.5
- new net ADC7: IC1.22, SV2.4
- new net N$25: R5.1, U1.1
- new net N$26: R6.1, U1.15
- net +12V: now also U1.4; no longer IC4.4
- net +5V: now also U1.9; no longer IC4.10, IC4.12, IC4.5, IC4.7, IC4.9
- net ENA: now also U1.6; no longer IC4.6
- net ENB: now also U1.11; no longer IC4.11
- net GND: now also U1.12, U1.7, U1.8; no longer IC4.8
- net OUT1: now also U1.2; no longer IC4.2
- net OUT2: now also U1.3; no longer IC4.3
- net OUT3: now also U1.13; no longer IC4.13
- net OUT4: now also U1.14; no longer IC4.14
- net PC4: no longer SV2.5
- net PC5: no longer SV2.4
- net PD3: now also U1.10
- net PD4: no longer R8.1
- net PD6: now also R8.1
- net PD7: now also U1.5
Routing:
- net ADC6: track 0.00 -> 42.7 mm, vias 0 -> 2
- net PC4: track 37.0 -> 0.00 mm, vias 2 -> 0
- net ADC7: track 0.00 -> 35.2 mm, vias 0 -> 2
- net PC5: track 32.6 -> 0.00 mm, vias 2 -> 0
- net +5V: track 303.2 -> 283.7 mm
- net SEN_B: track 19.2 -> 0.00 mm, vias 1 -> 0
- net OUT4: track 35.9 -> 22.3 mm
- net SEN_A: track 13.2 -> 0.00 mm
- net OUT1: track 74.1 -> 60.9 mm, vias 2 -> 1
- net ENA: track 44.2 -> 36.2 mm, vias 3 -> 2
- net N$25: track 0.00 -> 7.58 mm
- net GND: track 42.8 -> 35.9 mm
- net ENB: track 42.9 -> 37.3 mm
- net OUT2: track 53.9 -> 48.4 mm
- net +12V: track 128.2 -> 123.4 mm, vias 5 -> 4
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Other:
- board text removed: "<3"
- board text removed: "oshw"
